Commit message: Phase 1 cleanup: Remove debug logs, dead code, extract TCP calculation utility
- Removed ~20 debug console.log statements from IK, playback, and control hooks
- Deleted commented JointLabels component and stubbed forwardKinematics function
- Fixed speedPercentage bug (should use 'speed' from store)
- Extracted TCP calculation to shared lib/tcpCalculations.ts (eliminates 270 lines duplication)
- Consolidated CARTESIAN_AXES and IkAxisMask definitions
- Updated TargetTCPVisualizer, ActualTCPVisualizer, and kinematics.ts to use shared utility

File: public/urdf/PAROL6.urdf (robot description, URDF)
Before this commit: robot parol6, 8 links, 7 joints
Joints:
- joint L4: limit lower=-2 upper=2 effort=300 velocity=3 -> lower=-3.5 upper=0.5 effort=300 velocity=3
