Commit message: chore: replace console.log with logger, move control to root page
Frontend Cleanup:
- Replace 109 console.log statements with proper logger system
- Move /control page to root (remove redirect)
- Add .env.example template
- Delete old documentation files (HOW_TO_DEBUG_CRASHES.md, etc.)
- Update all components to use logger.debug() instead of console.log()
- Update hooks to use logger for debugging
- Update stores to use logger for state changes

Logger Integration:
- Use logger.debug() for debug messages (most cases)
- Use logger.error() for errors
- Use logger.warn() for warnings
- Proper source tags for all log messages

🤖 Generated with [Claude Code](https://claude.com/claude-code)

Co-Authored-By: Claude <noreply@anthropic.com>

File: public/urdf/PAROL6.urdf (robot description, URDF)
Before this commit: robot parol6, 8 links, 7 joints
Joints:
- joint L1: limit lower=-1.7 upper=1.7 effort=300 velocity=3 -> lower=-2.1475731 upper=2.1475731 effort=300 velocity=3; origin xyz=0 0 0 rpy=0 0 0 -> xyz=0 0 0.1105 rpy=0 0 0
- joint L2: limit lower=-0.98 upper=1 effort=300 velocity=3 -> lower=-2.530881 upper=-0.05890486 effort=300 velocity=3; origin xyz=0.0234207210610375 0 0.1105 rpy=-1.5707963267949 0 0 -> xyz=0.0234207210610375 0 0 rpy=-1.5707963267949 0 0
- joint L3: axis 0 0 -1 -> 0 0 1; limit lower=-2 upper=1.3 effort=300 velocity=3 -> lower=1.88261685 upper=5.02423568 effort=300 velocity=3; origin xyz=0 -0.18 0 rpy=3.1416 0 -1.5708 -> xyz=0.18 0 0 rpy=3.14159265358979 0 0
- joint L4: axis 0 0 -1 -> 0 0 1; limit lower=-3.5 upper=0.5 effort=300 velocity=3 -> lower=-1.8407944 upper=1.8407944 effort=300 velocity=3; origin xyz=0.0435 0 0 rpy=1.5707963267949 0 3.14159265358979 -> xyz=-0.0435 0.17635 0 rpy=1.5707963267949 0 0
- joint L5: axis 0 0 -1 -> 0 0 1; limit lower=-2.1 upper=2.1 effort=300 velocity=3 -> lower=-1.57079633 upper=1.57079633 effort=300 velocity=3; origin xyz=0 0 -0.17635 rpy=-1.5708 0 0 -> xyz=0 0 0 rpy=-1.5707963267949 0 0
- joint L6: axis 0 0 -1 -> 0 0 1; limit lower=-3.1 upper=3.1 effort=300 velocity=3 -> lower=0.0 upper=6.28318531 effort=300 velocity=3; origin xyz=0 0 0 rpy=1.5708 0 0 -> xyz=0 0.0628 0 rpy=1.5707963267949 0 0; type continuous -> revolute
